Commit message: feat: change aichallenge gym ros

File: launch/ego_racecar.xacro (robot description, xacro)
@@ -1,107 +1,21 @@
 <?xml version="1.0"?>
 <!-- A simple model of the racecar for rviz -->
-<robot xmlns:xacro="http://www.ros.org/wiki/xacro" name="racecar">
-  <xacro:property name="wheelbase" value="0.3302" />
-  <xacro:property name="width" value="0.2032" />
-  <xacro:property name="height" value="0.1" />
-  <xacro:property name="ground_offset" value="0.04" />
-  <xacro:property name="wheel_radius" value="0.0508" />
-  <xacro:property name="wheel_length" value="0.0381" />
-  <xacro:property name="laser_distance_from_base_link" value="0.275" />
-  <xacro:property name="laser_height" value="0.05" />
-  <xacro:property name="laser_radius" value="0.026" />
-  <xacro:property name="car_name" value="ego_racecar" />
-  <material name="black">
-    <color rgba="0.2 0.2 0.2 1."/>
-  </material>
-  <material name="blue">
-    <color rgba="0.3 0.57 1. 1."/>
-  </material>
-  <link name="${car_name}/base_link">
+<robot xmlns:xacro="http://ros.org/wiki/xacro" name="racecar">
+  <xacro:property name="wheel_radius" value="0.24" />           <!-- ホイール半径 -->
+  <xacro:property name="wheel_width" value="0.18" />            <!-- 後輪の幅 -->
+  <xacro:property name="wheel_base" value="1.087" />            <!-- ホイールベース（前後中心間） -->
+  <xacro:property name="wheel_tread" value="1.12" />            <!-- トレッド（後輪左右中心間） -->
+  <xacro:property name="front_overhang" value="0.467" />        <!-- フロントオーバーハング -->
+  <xacro:property name="rear_overhang" value="0.510" />         <!-- リアオーバーハング -->
+  <xacro:property name="left_overhang" value="0.09" />          <!-- 左オーバーハング（後輪中心から車体左端まで） -->
+  <xacro:property name="right_overhang" value="0.09" />         <!-- 右オーバーハング（後輪中心から車体右端まで） -->
+  <xacro:property name="vehicle_height" value="2.2" />          <!-- 車両全高（センサ含む） -->
+  <xacro:property name="max_steer_angle" value="0.64" />        <!-- 最大操舵角 [rad] -->
+  <link name="base_link">
     <visual>
-      <origin xyz="${wheelbase/2} 0 ${ground_offset+height/2}"/>
+      <origin xyz="0 0 0" rpy="0 0 1.57"/>
       <geometry>
-        <box size="${wheelbase} ${width} ${height}"/>
+        <mesh filename="package://aichallenge_gym_ros/launch/kart.dae" scale="1 1 1"/>
       </geometry>
-      <material name="blue"/>
-    </visual>
-  </link>
-  <joint name="base_to_laser_model" type="fixed">
-    <parent link="${car_name}/base_link"/>
-    <child link="${car_name}/laser_model"/>
-    <origin xyz="${laser_distance_from_base_link} 0 ${ground_offset+height+(laser_height/2)}"/>
-  </joint>
-  <link name="${car_name}/laser_model">
-    <visual>
-      <geometry>
-        <cylinder radius="${laser_radius}" length="${laser_height}"/>
-      </geometry>
-      <material name="black"/>
-    </visual>
-  </link>
-  <joint name="$base_to_back_left_wheel" type="fixed">
-    <parent link="${car_name}/base_link"/>
-    <child link="${car_name}/back_left_wheel"/>
-    <origin xyz="0 ${(wheel_length+width)/2} ${wheel_radius}"/>
-  </joint>
-  <link name="${car_name}/back_left_wheel">
-    <visual>
-      <geometry>
-        <cylinder radius="${wheel_radius}" length="${wheel_length}"/>
-      </geometry>
-      <material name="black"/>
-      <origin rpy="${pi/2} 0 0"/>
-    </visual>
-  </link>
-  <joint name="base_to_back_right_wheel" type="fixed">
-    <parent link="${car_name}/base_link"/>
-    <child link="${car_name}/back_right_wheel"/>
-    <origin xyz="0 ${-(wheel_length+width)/2} ${wheel_radius}"/>
-  </joint>
-  <link name="${car_name}/back_right_wheel">
-    <visual>
-      <geometry>
-        <cylinder radius="${wheel_radius}" length="${wheel_length}"/>
-      </geometry>
-      <material name="black"/>
-      <origin rpy="${pi/2} 0 0"/>
-    </visual>
-  </link>
-  <joint name="base_to_front_left_hinge" type="fixed">
-    <parent link="${car_name}/base_link"/>
-    <child link="${car_name}/front_left_hinge"/>
-    <origin xyz="${wheelbase} ${(wheel_length+width)/2} ${wheel_radius}"/>
-  </joint>
-  <link name="${car_name}/front_left_hinge"/>
-  <joint name="front_left_hinge_to_wheel" type="continuous">
-    <parent link="${car_name}/front_left_hinge"/>
-    <child link="${car_name}/front_left_wheel"/>
-  </joint>
-  <link name="${car_name}/front_left_wheel">
-    <visual>
-      <geometry>
-        <cylinder radius="${wheel_radius}" length="${wheel_length}"/>
-      </geometry>
-      <material name="black"/>
-      <origin rpy="${pi/2} 0 0"/>
-    </visual>
-  </link>
-  <joint name="base_to_front_right_hinge" type="fixed">
-    <parent link="${car_name}/base_link"/>
-    <child link="${car_name}/front_right_hinge"/>
-    <origin xyz="${wheelbase} ${-(wheel_length+width)/2} ${wheel_radius}"/>
-  </joint>
-  <link name="${car_name}/front_right_hinge"/>
-  <joint name="front_right_hinge_to_wheel" type="continuous">
-    <parent link="${car_name}/front_right_hinge"/>
-    <child link="${car_name}/front_right_wheel"/>
-  </joint>
-  <link name="${car_name}/front_right_wheel">
-    <visual>
-      <geometry>
-        <cylinder radius="${wheel_radius}" length="${wheel_length}"/>
-      </geometry>
-      <material name="black"/>
-      <origin rpy="${pi/2} 0 0"/>
     </visual>
   </link>
